File: AmazonDash/AmazonDash.brd (EAGLE design)
At the start: 83.4 x 20.9 mm, 40 parts, among them U1 3.3V, U2 FT231XS, U3 MCP73831, U4 ATMEGA328P_TQFP, U5 RFM69HCW, U6 FDC6392S, Y1 8MHZ

Commit message: Adding Amazon Dash CAM files and added outline to schematic
Parts:
- added FRAME2: FRAME-LEDGER, SparkFun-Aesthetics:CREATIVE_COMMONS
Changed lines of the file:
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@@
 <grid distance="1" unitdist="mil" unit="mm" style="lines" multiple="1" display="yes" altdistance="0.025" altunitdist="inch" altunit="inch"/>
 <layers>
-<layer number="1" name="Top" color="4" fill="1" visible="yes" active="yes"/>
+<layer number="1" name="Top" color="4" fill="1" visible="no" active="yes"/>
 <layer number="2" name="Route2" color="1" fill="3" visible="no" active="no"/>
 <layer number="3" name="Route3" color="4" fill="3" visible="no" active="no"/>
 <layer number="14" name="Route14" color="1" fill="6" visible="no" active="no"/>
 <layer number="15" name="Route15" color="4" fill="6" visible="no" active="no"/>
-<layer number="16" name="Bottom" color="1" fill="1" visible="yes" active="yes"/>
-<layer number="17" name="Pads" color="2" fill="1" visible="yes" active="yes"/>
-<layer number="18" name="Vias" color="2" fill="1" visible="yes" active="yes"/>
+<layer number="16" name="Bottom" color="1" fill="1" visible="no" active="yes"/>
+<layer number="17" name="Pads" color="2" fill="1" visible="no" active="yes"/>
+<layer number="18" name="Vias" color="2" fill="1" visible="no" active="yes"/>
 <layer number="19" name="Unrouted" color="6" fill="1" visible="yes" active="yes"/>
 <layer number="20" name="Dimension" color="15" fill="1" visible="yes" active="yes"/>
@@
 <attribute name="NAME" x="46.3426" y="18.7494" size="1" layer="25" ratio="9" rot="R270"/>
 </element>
+<element name="FRAME2" library="SparkFun-Aesthetics" package="CREATIVE_COMMONS" value="FRAME-LEDGER" x="17.2466" y="-17.1704"/>
 </elements>
 <signals>
